File: Układ_mnożący.kicad_pcb (KiCad board)
At the start: 2 copper layers, 30 x 60 mm, 48 parts, among them IC1 LMC7660IM_NOPB, J1 Conn_01x02_Male, J2 Conn_01x01_Male, J3 Conn_01x01_Male, J4 Conn_01x01_Male, J5 Conn_01x01_Male, J6 Conn_01x01_Male, J7 Conn_01x01_Male, Q1 DMG1012UW, U1 TLC2272ACD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

Commit message: Final Electrical Schematic v2
Added pinout to Vref
Parts:
- added J8: Conn_01x01_Male, Connector_PinHeader_2.54mm:PinHeader_1x01_P2.54mm_Vertical, F.Cu at (99.8, 29.2)
Changed lines of the file:
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@@
+    )
+  )
+  (footprint "Connector_PinHeader_2.54mm:PinHeader_1x01_P2.54mm_Vertical" (layer "F.Cu")
+    (at 99.822 29.21)
+    (descr "Through hole straight pin header, 1x01, 2.54mm pitch, single row")
+    (tags "Through hole pin header THT 1x01 2.54mm single row")
+    (property "Sheetfile" "Plik: Układ_mnożący.kicad_sch")
+    (property "Sheetname" "")
+    (attr through_hole)
+    (fp_text reference "J8" (at 0 -2.33) (layer "F.SilkS")
+      (effects (font (size 1 1) (thickness 0.15)))
+    )
+    (fp_text value "Conn_01x01_Male" (at 0 2.33) (layer "F.Fab")
+      (effects (font (size 1 1) (thickness 0.15)))
+    )
+    (fp_text user "${REFERENCE}" (at 0 0 90) (layer "F.Fab")
+      (effects (font (size 1 1) (thickness 0.15)))
+    )
+    (fp_line (start -1.33 -1.33) (end 0 -1.33) (layer "F.SilkS") (width 0.12))
+    (fp_line (start -1.33 1.33) (end 1.33 1.33) (layer "F.SilkS") (width 0.12))
+    (fp_line (start -1.33 1.27) (end 1.33 1.27) (layer "F.SilkS") (width 0.12))
+    (fp_line (start -1.33 1.27) (end -1.33 1.33) (layer "F.SilkS") (width 0.12))
+    (fp_line (start -1.33 0) (end -1.33 -1.33) (layer "F.SilkS") (width 0.12))
+    (fp_line (start 1.33 1.27) (end 1.33 1.33) (layer "F.SilkS") (width 0.12))
+    (fp_line (start -1.8 1.8) (end 1.8 1.8) (layer "F.CrtYd") (width 0.05))
+    (fp_line (start 1.8 1.8) (end 1.8 -1.8) (layer "F.CrtYd") (width 0.05))
+    (fp_line (start 1.8 -1.8) (end -1.8 -1.8) (layer "F.CrtYd") (width 0.05))
+    (fp_line (start -1.8 -1.8) (end -1.8 1.8) (layer "F.CrtYd") (width 0.05))
+    (fp_line (start -1.27 1.27) (end -1.27 -0.635) (layer "F.Fab") (width 0.1))
+    (fp_line (start -1.27 -0.635) (end -0.635 -1.27) (layer "F.Fab") (width 0.1))
+    (fp_line (start -0.635 -1.27) (end 1.27 -1.27) (layer "F.Fab") (width 0.1))
+    (fp_line (start 1.27 1.27) (end -1.27 1.27) (layer "F.Fab") (width 0.1))
+    (fp_line (start 1.27 -1.27) (end 1.27 1.27) (layer "F.Fab") (width 0.1))
+    (pad "1" thru_hole rect (at 0 0) (size 1.7 1.7) (drill 1) (layers *.Cu *.Mask)
+      (net 23 "Vref") (pinfunction "Pin_1") (pintype "passive"))
+    (model "${KICAD6_3DMODEL_DIR}/Connector_PinHeader_2.54mm.3dshapes/PinHeader_1x01_P2.54mm_Vertical.wrl"
+      (offset (xyz 0 0 0))
+      (scale (xyz 1 1 1))
+      (rotate (xyz 0 0 0))
     )
   )

Commit message: Final PCB design
Parts:
- C3, C5: footprint Capacitor_THT:CP_Radial_D5.0mm_P2.50mm -> Capacitor_SMD:C_1206_3216Metric_Pad1.33x1.80mm_HandSolder
- C6: footprint Capacitor_SMD:C_1206_3216Metric_Pad1.33x1.80mm_HandSolder -> Capacitor_Tantalum_SMD:CP_EIA-3528-21_Kemet-B
- J1: value Conn_01x02_Male -> Conn_01x01_Male; footprint Connector_PinHeader_2.54mm:PinHeader_1x02_P2.54mm_Vertical -> Connector_PinHeader_2.54mm:PinHeader_1x01_P2.54mm_Vertical
- J3: value Conn_01x01_Male -> Conn_01x02_Male; footprint Connector_PinHeader_2.54mm:PinHeader_1x01_P2.54mm_Vertical -> Connector_PinHeader_2.54mm:PinHeader_1x02_P2.54mm_Vertical
- moved R8 84.9 mm to (30.2, 48.8), turned to -90 degrees
- moved J4 83.8 mm to (41.1, 28.4)
- moved R13 82.5 mm to (32.5, 67.3), turned to -90 degrees
- moved C10 82.2 mm to (36.3, 50.8), turned to 180 degrees
- moved C13 80.6 mm to (36.6, 72.1), turned to 180 degrees
- moved R11 79.7 mm to (30.0, 71.4), turned to 90 degrees
- moved R7 78.9 mm to (30.2, 38.1), turned to -90 degrees
- moved J7 78.8 mm to (41.9, 73.2)
- moved C14 77.9 mm to (36.3, 61.5), turned to 180 degrees
- moved J6 75.7 mm to (47.2, 48.5)
- moved RV1 75.6 mm to (22.6, 40.9)
- moved J5 75.0 mm to (43.4, 44.7)
- moved C15 74.7 mm to (39.4, 53.8)
- moved J1 73.6 mm to (31.5, 45.0)
- moved C8 72.6 mm to (36.3, 40.1), turned to 180 degrees
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Connections:
- J3 pad 1: Vcc -> GND
- J8 pad 1: Vref -> Vx
- RV1 pad 3: Vref -> unconnected-(RV1-Pad3)
- RV2 pad 3: V1 -> unconnected-(RV2-Pad3)
- RV3 pad 1: Net-(R8-Pad2) -> unconnected-(RV3-Pad1)
- RV4 pad 3: Net-(R10-Pad1) -> unconnected-(RV4-Pad3)
Routing:
- net 4V2: track 0.00 -> 93.4 mm
- net -4V2: track 0.00 -> 57.8 mm
- net Net-(C7-Pad1): track 0.00 -> 45.8 mm
- net V4: track 0.00 -> 31.4 mm
- net V1: track 0.00 -> 29.4 mm
- net Net-(R11-Pad1): track 0.00 -> 28.7 mm
- net V2: track 0.00 -> 24.5 mm, vias 0 -> 2
- net Vref: track 0.00 -> 23.2 mm
- net Net-(R11-Pad2): track 0.00 -> 20.3 mm
- net Net-(R6-Pad2): track 0.00 -> 19.6 mm, vias 0 -> 2
- net Net-(R8-Pad2): track 0.00 -> 17.6 mm, vias 0 -> 1
- net V3: track 0.00 -> 17.4 mm
- net Net-(Q1-Pad1): track 0.00 -> 11.4 mm
- net Vcc: track 0.00 -> 10.5 mm
- net Net-(R1-Pad2): track 0.00 -> 8.86 mm
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- added copper zone on B.Cu, net GND
- added copper zone on F.Cu, net GND

Commit message: Final PCB design v2
Parts:
- added J9: Conn_01x01_Male, Connector_PinHeader_2.54mm:PinHeader_1x01_P2.54mm_Vertical, F.Cu at (24.6, 49.5)
- moved J4 16.9 mm to (45.7, 44.7)
- moved J2 14.4 mm to (35.1, 77.7)
- moved RV4 10.4 mm to (44.5, 67.5)
- moved C12 9.96 mm to (33.5, 72.4), turned to 180 degrees
- moved R12 9.08 mm to (29.7, 62.7), turned to -90 degrees
- moved R11 9.00 mm to (27.4, 62.7), turned to -90 degrees
- moved R13 7.79 mm to (35.1, 74.7), turned to 180 degrees
- moved C7 7.42 mm to (42.4, 70.9), turned to -90 degrees
- moved RV2 7.37 mm to (47.6, 40.6)
- moved C13 7.37 mm to (36.6, 64.8), turned to 0 degrees
- moved R10 4.75 mm to (40.1, 70.9), turned to -90 degrees
- moved R1 3.88 mm to (42.4, 40.2)
- moved R2 3.88 mm to (42.4, 36.1)
- moved J7 3.78 mm to (45.5, 71.9)
- moved C2 3.64 mm to (29.2, 37.3), turned to 0 degrees
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Connections:
- C12 pad 2: -4V2 -> 4V2
- C13 pad 2: 4V2 -> -4V2
- U5 pad 4: 4V2 -> -4V2
- U5 pad 8: -4V2 -> 4V2
Routing:
- net V1: track 29.4 -> 15.3 mm
- net Net-(R11-Pad1): track 28.7 -> 14.7 mm
- net Net-(C7-Pad1): track 45.8 -> 33.3 mm, vias 0 -> 2
- net Net-(R13-Pad2): track 5.91 -> 17.4 mm
- net V4: track 31.4 -> 20.5 mm
- net Net-(R11-Pad2): track 20.3 -> 11.9 mm
- net Net-(R6-Pad2): track 19.6 -> 26.6 mm
- net 4V2: track 93.4 -> 90.1 mm
- net Net-(Q1-Pad1): track 11.4 -> 8.50 mm
- net Vout: track 5.97 -> 8.42 mm
- net Vref: track 23.2 -> 24.8 mm
- net Net-(R1-Pad2): track 8.86 -> 7.43 mm
- net V3: track 17.4 -> 18.6 mm
- net Net-(R10-Pad1): track 6.82 -> 5.62 mm
- net V2: track 24.5 -> 23.3 mm
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